Commit message: 更新 rm_arm_2025_last.urdf，添加关节限制的努力和速度参数

File: rm_arm_2025_last/urdf/rm_arm_2025_last.urdf (robot description, URDF)
Before this commit: robot rm_arm_2025_last, 7 links, 6 joints
Joints:
- joint joint1: limit (none) -> effort=1000 velocity=3.14
- joint joint2: limit lower=-2.4 upper=2.4 effort=0 velocity=0 -> lower=-2.4 upper=2.4 effort=1000 velocity=3.14
- joint joint3: limit lower=-2.4 upper=2.4 effort=0 velocity=0 -> lower=-2.4 upper=2.4 effort=1000 velocity=3.14
- joint joint4: limit (none) -> effort=1000 velocity=3.14
- joint joint5: limit lower=-1.74 upper=1.74 effort=0 velocity=0 -> lower=-1.74 upper=1.74 effort=1000 velocity=3.14
- joint joint6: limit (none) -> effort=1000 velocity=3.14
